Commit message: Enhance Delivery Manager and Obstacle Detector for improved functionality
- Refactored DeliveryManager to use one-shot timers for loading and unloading processes, preventing repeated callbacks.
- Introduced new methods `_on_loading_timer` and `_on_unloading_timer` for better timer management.
- Enhanced ObstacleDetector with advanced tracking capabilities, including temporal history for obstacles and spatial indexing for efficient clustering.
- Updated obstacle classification to better suit Ethiopian urban environments, with new categories and size thresholds.
- Improved visualization markers for obstacles, including velocity indicators and category labels.
- Adjusted navigation parameters in nav2_params.yaml for safer urban navigation, including reduced velocity thresholds and inflation layer settings.

File: medbot_ws/src/medbot_description/urdf/robot_core.xacro (robot description, xacro)
@@ -31,4 +31,5 @@
   <xacro:macro name="box_inertia" params="m w h d">
     <inertial>
+      <origin xyz="0 0 0" rpy="0 0 0"/>
       <mass value="${m}"/>
       <inertia ixx="${(m/12)*(h*h+d*d)}" ixy="0" ixz="0"
@@ -39,4 +40,5 @@
   <xacro:macro name="cylinder_inertia" params="m r h">
     <inertial>
+      <origin xyz="0 0 0" rpy="0 0 0"/>
       <mass value="${m}"/>
       <inertia ixx="${(m/12)*(3*r*r+h*h)}" ixy="0" ixz="0"
@@ -47,4 +49,5 @@
   <xacro:macro name="sphere_inertia" params="m r">
     <inertial>
+      <origin xyz="0 0 0" rpy="0 0 0"/>
       <mass value="${m}"/>
       <inertia ixx="${(2/5)*m*r*r}" ixy="0" ixz="0"

File: medbot_ws/src/medbot_description/urdf/sensors/camera.xacro (robot description, xacro)
@@ -27,4 +27,5 @@
       </collision>
       <inertial>
+        <origin xyz="0 0 0" rpy="0 0 0"/>
         <mass value="${camera_mass}"/>
         <inertia ixx="${(camera_mass/12)*(camera_size*camera_size*5)}" ixy="0" ixz="0"

File: medbot_ws/src/medbot_description/urdf/sensors/imu.xacro (robot description, xacro)
@@ -27,4 +27,5 @@
       </collision>
       <inertial>
+        <origin xyz="0 0 0" rpy="0 0 0"/>
         <mass value="${imu_mass}"/>
         <inertia ixx="${(imu_mass/12)*(imu_size*imu_size*2)}" ixy="0" ixz="0"

File: medbot_ws/src/medbot_description/urdf/sensors/lidar.xacro (robot description, xacro)
@@ -28,4 +28,5 @@
       </collision>
       <inertial>
+        <origin xyz="0 0 0" rpy="0 0 0"/>
         <mass value="${lidar_mass}"/>
         <inertia ixx="${(lidar_mass/12)*(3*lidar_radius*lidar_radius+lidar_height*lidar_height)}"
